Commit message: small fix

File: urdf/wall.xacro (robot description, xacro)
@@ -30,5 +30,5 @@
   </link>
     <gazebo reference="wall_${name}_link">
-    <material>Gazebo/"${color}</material>
+    <material>Gazebo/Red</material>
   </gazebo>
   </xacro:macro>

Commit message: Changed definition of origin of wall from bottom center to the center of volume.

File: urdf/wall.xacro (robot description, xacro)
@@ -1,7 +1,5 @@
 <?xml version="1.0"?>
 <robot xmlns:xacro="http://www.ros.org/wiki/xacro">
-  <xacro:property name="width" value=".5" />
-  <xacro:property name="height" value="4" />
- <xacro:macro name="wall" params="name mass len *origin">
+ <xacro:macro name="wall" params="name mass width height len *origin">
     <joint name="world_${name}_joint" type="fixed">
       <xacro:insert_block name="origin"/>
@@ -11,10 +9,10 @@
     <link name="wall_${name}_link">
     <inertial>
-      <origin xyz="0 ${width/2} ${height/2}" />
+      <origin xyz="0 0 ${height/2}" />
       <mass value="${mass}" />
       <inertia  ixx="1.0" ixy="0.0"  ixz="0.0"  iyy="100.0"  iyz="0.0"  izz="1.0" />
     </inertial>
     <visual>
-      <origin xyz="0 ${width/2} ${height/2}"/>
+      <origin xyz="0 0 ${height/2}"/>
       <geometry>
         <box size="${len} ${width} ${height}" />
@@ -23,5 +21,5 @@
     </visual>
     <collision>
-      <origin xyz="0 ${width/2} ${height/2}"/>
+      <origin xyz="0 0 ${height/2}"/>
       <geometry>
         <box size="${len} ${width} ${height}" />
